File: NeopixelMatrix.kicad_sch (KiCad schematic)
At the start: 304 parts

Commit message: Version 2
Parts:
- added R8 (x7): 0, Resistor_SMD:R_0402_1005Metric, symbol Device:R_US
- C6: footprint Capacitor_SMD:C_0402_1005Metric -> Capacitor_SMD:C_0603_1608Metric
Connections:
- net STRIP10 is gone; now on net END-STRIP19: N163.4 (DIN)
- net STRIP12 is gone; now on net END-STRIP11: N199.4 (DIN)
- net STRIP14 is gone; now on net END-STRIP13: N235.4 (DIN)
- net STRIP16 is gone; now on net END-STRIP15: N271.4 (DIN)
- net STRIP2 is gone; now on net END-STRIP1: N19.4 (DIN)
- net STRIP4 is gone; now on net END-STRIP3: N55.4 (DIN)
- net STRIP6 is gone; now on net END-STRIP5: N91.4 (DIN)
- net STRIP8 is gone; now on net END-STRIP7: N127.4 (DIN)
- net END-STRIP10: now also R8.1
- net END-STRIP12: now also R8.1
- net END-STRIP14: now also R8.1
- net END-STRIP2: now also R8.1
- net END-STRIP4: now also R8.1
- net END-STRIP6: now also R8.1
- net END-STRIP8: now also R8.1
- net STRIP11: now also R8.2
- net STRIP13: now also R8.2
- net STRIP15: now also R8.2
- net STRIP3: now also R8.2
- net STRIP5: now also R8.2
- net STRIP7: now also R8.2
- net STRIP9: now also R8.2

Commit message: V3 update in preparation for sale
Parts:
- removed C6 (x16): 10uF, Capacitor_SMD:C_0603_1608Metric, symbol Device:C
- removed R8 (x7): 0, Resistor_SMD:R_0402_1005Metric, symbol Device:R_US
- N1, N10, N100, N101, N102, N103, N104, N105, N106, N107, N108, N109, N11, N110, N111, N112, N113, N114, N115, N116, N117, N118, N119, N12, N120, N121, N122, N123, N124, N125, N126, N127, N128, N129, N13, N130, N131, N132, N133, N134, N135, N136, N137, N138, N139, N14, N140, N141, N142, N143, N144, N145, N146, N147, N148, N149, N15, N150, N151, N152, N153, N154, N155, N156, N157, N158, N159, N16, N160, N161, N162, N163, N164, N165, N166, N167, N168, N169, N17, N170, N171, N172, N173, N174, N175, N176, N177, N178, N179, N18, N180, N181, N182, N183, N184, N185, N186, N187, N188, N189, N19, N190, N191, N192, N193, N194, N195, N196, N197, N198, N199, N2, N20, N200, N201, N202, N203, N204, N205, N206, N207, N208, N209, N21, N210, N211, N212, N213, N214, N215, N216, N217, N218, N219, N22, N220, N221, N222, N223, N224, N225, N226, N227, N228, N229, N23, N230, N231, N232, N233, N234, N235, N236, N237, N238, N239, N24, N240, N241, N242, N243, N244, N245, N246, N247, N248, N249, N25, N250, N251, N252, N253, N254, N255, N256, N257, N258, N259, N26, N260, N261, N262, N263, N264, N265, N266, N267, N268, N269, N27, N270, N271, N272, N273, N274, N275, N276, N277, N278, N279, N28, N280, N281, N282, N283, N284, N285, N286, N287, N288, N29, N3, N30, N31, N32, N33, N34, N35, N36, N37, N38, N39, N4, N40, N41, N42, N43, N44, N45, N46, N47, N48, N49, N5, N50, N51, N52, N53, N54, N55, N56, N57, N58, N59, N6, N60, N61, N62, N63, N64, N65, N66, N67, N68, N69, N7, N70, N71, N72, N73, N74, N75, N76, N77, N78, N79, N8, N80, N81, N82, N83, N84, N85, N86, N87, N88, N89, N9, N90, N91, N92, N93, N94, N95, N96, N97, N98, N99: value ~ -> SK6805-EC14; LCSC Part # (none) -> C2909055
